File: pcb/pump.kicad_sch (KiCad schematic)
At the start: 8 parts, among them IC4 DRV8837CDSGR

Commit message: created step file
Parts:
- removed C12, C13: 10u, Capacitor_SMD:C_0805_2012Metric, symbol Capacitor_JLC:10u
- added C8, C9: 10u_0402, Capacitor_SMD:C_0402_1005Metric, symbol Capacitor_JLC:10u_0402
Connections:
- net GND: now also C8.2, C9.2
- net VBUS: now also C8.1, C9.1
Changed lines of the file:
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@@
-    (stroke (width 0) (type default))
-  )
-  (wire (pts (xy 272.415 153.67) (xy 272.415 156.21))
     (stroke (width 0) (type default))
   )
@@
     (stroke (width 0) (type default))
   )
+  (wire (pts (xy 260.985 156.21) (xy 277.495 156.21))
+    (stroke (width 0) (type default))
+  )
   (wire (pts (xy 336.55 165.1) (xy 336.55 167.005))
     (stroke (width 0) (type default))
@@
     (stroke (width 0) (type default))
   )
-  (wire (pts (xy 272.415 144.78) (xy 260.985 144.78))
-    (stroke (width 0) (type default))
-  )
-  (wire (pts (xy 272.415 156.21) (xy 260.985 156.21))
-    (stroke (width 0) (type default))
-  )
   (wire (pts (xy 233.045 162.56) (xy 260.985 162.56))
     (stroke (width 0) (type default))
@@
     (stroke (width 0) (type default))
   )
+  (wire (pts (xy 277.495 153.67) (xy 277.495 156.21))
+    (stroke (width 0) (type default))
+  )
   (polyline (pts (xy 285.496 180.594) (xy 170.688 180.594))
     (stroke (width 0) (type default))
   )
-  (wire (pts (xy 272.415 146.05) (xy 272.415 144.78))
+  (wire (pts (xy 277.495 146.05) (xy 277.495 144.78))
     (stroke (width 0) (type default))
   )
@@
   )
   (polyline (pts (xy 370.205 113.665) (xy 370.205 180.34))
+    (stroke (width 0) (type default))
+  )
+  (wire (pts (xy 260.985 144.78) (xy 277.495 144.78))
     (stroke (width 0) (type default))
   )
@@
     (pin "1")
     (instances
-      (project "Grower"
+      (project "PlantBot"
         (path "/1fa508ef-df83-4c99-846b-9acf535b3ad9/11ddc7da-b07f-4cec-87b3-82aa721f8223"
           (reference "#PWR0122") (unit 1)
-        )
-      )
-    )
-  )
-  (symbol (lib_id "Capacitor_JLC:10u") (at 260.985 149.86 0) (unit 1)
-    (in_bom yes) (on_board yes) (dnp no) (fields_autoplaced)
-    (property "Reference" "C12" (at 263.906 146.1764 0)
-      (effects (font (size 1.27 1.27)) (justify left))
-    )
-    (property "Value" "10u" (at 263.906 148.9515 0)
-      (effects (font (size 1.27 1.27)) (justify left))
-    )
-    (property "Footprint" "Capacitor_SMD:C_0805_2012Metric" (at 261.9502 153.67 0)
-      (effects (font (size 1.27 1.27)) hide)
-    )
-    (property "Datasheet" "~" (at 260.985 149.86 0)
-      (effects (font (size 1.27 1.27)) hide)
-    )
-    (property "Type" "X5R" (at 263.906 151.7266 0)
-      (effects (font (size 1.27 1.27)) (justify left))
-    )
-    (property "LCSC" "C15850" (at 260.985 149.86 0)
-      (effects (font (size 1.27 1.27)) hide)
-    )
-    (property "Voltage" "25V" (at 263.906 154.5017 0)
-      (effects (font (size 1.27 1.27)) (justify left))
-    )
-    (pin "1")
-    (pin "2")
-    (instances
-      (project "Grower"
-        (path "/1fa508ef-df83-4c99-846b-9acf535b3ad9/11ddc7da-b07f-4cec-87b3-82aa721f8223"
-          (reference "C12") (unit 1)
         )
       )
@@
     (pin "9")
     (instances
-      (project "Grower"
+      (project "PlantBot"
         (path "/1fa508ef-df83-4c99-846b-9acf535b3ad9/11ddc7da-b07f-4cec-87b3-82aa721f8223"
           (reference "IC4") (unit 1)
@@
     (pin "1")
     (instances
-      (project "Grower"
+      (project "PlantBot"
         (path "/1fa508ef-df83-4c99-846b-9acf535b3ad9/11ddc7da-b07f-4cec-87b3-82aa721f8223"
           (reference "#PWR0129") (unit 1)
@@
     (pin "2")
     (instances
-      (project "Grower"
+      (project "PlantBot"
         (path "/1fa508ef-df83-4c99-846b-9acf535b3ad9/11ddc7da-b07f-4cec-87b3-82aa721f8223"
           (reference "C11") (unit 1)
@@
     )
   )
-  (symbol (lib_id "Capacitor_JLC:10u") (at 272.415 149.86 0) (unit 1)
-    (in_bom yes) (on_board yes) (dnp no) (fields_autoplaced)
-    (property "Reference" "C13" (at 275.336 146.1764 0)
-      (effects (font (size 1.27 1.27)) (justify left))
-    )
-    (property "Value" "10u" (at 275.336 148.9515 0)
-      (effects (font (size 1.27 1.27)) (justify left))
-    )
-    (property "Footprint" "Capacitor_SMD:C_0805_2012Metric" (at 273.3802 153.67 0)
-      (effects (font (size 1.27 1.27)) hide)
-    )
-    (property "Datasheet" "~" (at 272.415 149.86 0)
-      (effects (font (size 1.27 1.27)) hide)
-    )
-    (property "Type" "X5R" (at 275.336 151.7266 0)
-      (effects (font (size 1.27 1.27)) (justify left))
-    )
-    (property "LCSC" "C15850" (at 272.415 149.86 0)
-      (effects (font (size 1.27 1.27)) hide)
-    )
-    (property "Voltage" "25V" (at 275.336 154.5017 0)
-      (effects (font (size 1.27 1.27)) (justify left))
-    )
-    (pin "1")
-    (pin "2")
-    (instances
-      (project "Grower"
-        (path "/1fa508ef-df83-4c99-846b-9acf535b3ad9/11ddc7da-b07f-4cec-87b3-82aa721f8223"
-          (reference "C13") (unit 1)
-        )
-      )
-    )
-  )
   (symbol (lib_id "power:GND") (at 180.975 146.05 0) (unit 1)
     (in_bom yes) (on_board yes) (dnp no)
@@
     (pin "1")
     (instances
-      (project "Grower"
+      (project "PlantBot"
         (path "/1fa508ef-df83-4c99-846b-9acf535b3ad9/11ddc7da-b07f-4cec-87b3-82aa721f8223"
           (reference "#PWR0131") (unit 1)
@@
     (pin "2")
     (instances
-      (project "Grower"
+      (project "PlantBot"
         (path "/1fa508ef-df83-4c99-846b-9acf535b3ad9/11ddc7da-b07f-4cec-87b3-82aa721f8223"
           (reference "D9") (unit 1)
@@
     (pin "1")
     (instances
-      (project "Grower"
+      (project "PlantBot"
         (path "/1fa508ef-df83-4c99-846b-9acf535b3ad9/11ddc7da-b07f-4cec-87b3-82aa721f8223"
           (reference "#PWR0130") (unit 1)
@@
     (pin "2")
     (instances
-      (project "Grower"
+      (project "PlantBot"
         (path "/1fa508ef-df83-4c99-846b-9acf535b3ad9/11ddc7da-b07f-4cec-87b3-82aa721f8223"
           (reference "R29") (unit 1)
+        )
+      )
+    )
+  )
+  (symbol (lib_id "Capacitor_JLC:10u_0402") (at 260.985 149.86 0) (unit 1)
+    (in_bom yes) (on_board yes) (dnp no) (fields_autoplaced)
+    (property "Reference" "C8" (at 263.906 147.2953 0)
+      (effects (font (size 1.27 1.27)) (justify left))
+    )
+    (property "Value" "10u_0402" (at 263.906 149.2163 0)
+      (effects (font (size 1.27 1.27)) (justify left))
+    )
+    (property "Footprint" "Capacitor_SMD:C_0402_1005Metric" (at 293.37 151.765 0)
+      (effects (font (size 1.27 1.27)) hide)
+    )
+    (property "Datasheet" "~" (at 260.985 149.86 0)
+      (effects (font (size 1.27 1.27)) hide)
+    )
+    (property "Type" "X5R" (at 263.906 151.1373 0)
+      (effects (font (size 1.27 1.27)) (justify left))
+    )
+    (property "LCSC" "C315248" (at 280.67 149.86 0)
+      (effects (font (size 1.27 1.27)) hide)
+    )
+    (property "Voltage" "10V" (at 263.906 153.0583 0)
+      (effects (font (size 1.27 1.27)) (justify left))
+    )
+    (pin "1")
+    (pin "2")
+    (instances
+      (project "PlantBot"
+        (path "/1fa508ef-df83-4c99-846b-9acf535b3ad9/11ddc7da-b07f-4cec-87b3-82aa721f8223"
+          (reference "C8") (unit 1)
         )
       )
@@
     (pin "2")
     (instances
-      (project "Grower"
+      (project "PlantBot"
         (path "/1fa508ef-df83-4c99-846b-9acf535b3ad9/11ddc7da-b07f-4cec-87b3-82aa721f8223"
           (reference "R30") (unit 1)
@@
     (pin "1")
     (instances
-      (project "Grower"
+      (project "PlantBot"
         (path "/1fa508ef-df83-4c99-846b-9acf535b3ad9/11ddc7da-b07f-4cec-87b3-82aa721f8223"
           (reference "#PWR0144") (unit 1)
@@
     (pin "2")
     (instances
-      (project "Grower"
+      (project "PlantBot"
         (path "/1fa508ef-df83-4c99-846b-9acf535b3ad9/11ddc7da-b07f-4cec-87b3-82aa721f8223"
           (reference "D7") (unit 1)
@@
     )
   )
+  (symbol (lib_id "Capacitor_JLC:10u_0402") (at 277.495 149.86 0) (unit 1)
+    (in_bom yes) (on_board yes) (dnp no) (fields_autoplaced)
+    (property "Reference" "C9" (at 280.416 147.2953 0)
+      (effects (font (size 1.27 1.27)) (justify left))
+    )
+    (property "Value" "10u_0402" (at 280.416 149.2163 0)
+      (effects (font (size 1.27 1.27)) (justify left))
+    )
+    (property "Footprint" "Capacitor_SMD:C_0402_1005Metric" (at 309.88 151.765 0)
+      (effects (font (size 1.27 1.27)) hide)
+    )
+    (property "Datasheet" "~" (at 277.495 149.86 0)
+      (effects (font (size 1.27 1.27)) hide)
+    )
+    (property "Type" "X5R" (at 280.416 151.1373 0)
+      (effects (font (size 1.27 1.27)) (justify left))
+    )
+    (property "LCSC" "C315248" (at 297.18 149.86 0)
+      (effects (font (size 1.27 1.27)) hide)
+    )
+    (property "Voltage" "10V" (at 280.416 153.0583 0)
+      (effects (font (size 1.27 1.27)) (justify left))
+    )
+    (pin "1")
+    (pin "2")
+    (instances
+      (project "PlantBot"
+        (path "/1fa508ef-df83-4c99-846b-9acf535b3ad9/11ddc7da-b07f-4cec-87b3-82aa721f8223"
+          (reference "C9") (unit 1)
+        )
+      )
+    )
+  )
   (symbol (lib_id "power:GND") (at 260.985 162.56 0) (unit 1)
     (in_bom yes) (on_board yes) (dnp no)
@@
     (pin "1")
     (instances
-      (project "Grower"
+      (project "PlantBot"
         (path "/1fa508ef-df83-4c99-846b-9acf535b3ad9/11ddc7da-b07f-4cec-87b3-82aa721f8223"
           (reference "#PWR0128") (unit 1)
