File: pcb/PlantBot.kicad_sch (KiCad schematic)
At the start: 1 part

Commit message: created step file
Parts:
- removed FID1: Fiducial, personal:Product Stamp, symbol Mechanical:Fiducial
Other:
- sheet Microcontroller ports: added LIGHT_PWR; removed AMP_MIC_OUT, LIGHT_MIC_PWR, SCL, SDA, STH20_PWR
- sheet Sensor ports: added LIGHT_PWR; removed AMP_MIC_OUT, LIGHT_MIC_PWR, SCL, SDA, SHT20_PWR
Changed lines of the file:
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@@
     (rev "E")
   )
+  (wire (pts (xy 148.59 107.315) (xy 148.59 151.13))
+    (stroke (width 0) (type default))
+  )
   (wire (pts (xy 150.495 109.22) (xy 150.495 153.035))
     (stroke (width 0) (type default))
@@
     (stroke (width 0) (type default))
   )
-  (wire (pts (xy 147.955 105.41) (xy 147.955 147.955))
-    (stroke (width 0) (type default))
-  )
-  (wire (pts (xy 134.62 135.255) (xy 134.62 101.6))
-    (stroke (width 0) (type default))
-  )
-  (wire (pts (xy 147.955 147.955) (xy 116.84 147.955))
-    (stroke (width 0) (type default))
-  )
   (wire (pts (xy 161.29 109.22) (xy 150.495 109.22))
     (stroke (width 0) (type default))
   )
-  (wire (pts (xy 161.29 105.41) (xy 147.955 105.41))
-    (stroke (width 0) (type default))
-  )
-  (wire (pts (xy 149.225 151.13) (xy 149.225 107.315))
-    (stroke (width 0) (type default))
-  )
-  (wire (pts (xy 116.84 151.13) (xy 149.225 151.13))
+  (wire (pts (xy 161.29 107.315) (xy 148.59 107.315))
+    (stroke (width 0) (type default))
+  )
+  (wire (pts (xy 148.59 151.13) (xy 116.84 151.13))
     (stroke (width 0) (type default))
   )
@@
     (stroke (width 0) (type default))
   )
-  (wire (pts (xy 132.08 133.35) (xy 116.84 133.35))
-    (stroke (width 0) (type default))
-  )
   (wire (pts (xy 214.63 111.125) (xy 250.19 111.125))
     (stroke (width 0) (type default))
@@
     (stroke (width 0) (type default))
   )
-  (wire (pts (xy 161.29 99.695) (xy 132.08 99.695))
-    (stroke (width 0) (type default))
-  )
   (wire (pts (xy 337.82 89.535) (xy 337.82 143.51))
     (stroke (width 0) (type default))
   )
-  (wire (pts (xy 116.84 131.445) (xy 129.54 131.445))
-    (stroke (width 0) (type default))
-  )
-  (wire (pts (xy 129.54 97.79) (xy 129.54 131.445))
-    (stroke (width 0) (type default))
-  )
   (wire (pts (xy 337.82 143.51) (xy 331.47 143.51))
     (stroke (width 0) (type default))
   )
-  (wire (pts (xy 161.29 97.79) (xy 129.54 97.79))
-    (stroke (width 0) (type default))
-  )
   (wire (pts (xy 150.495 153.035) (xy 116.84 153.035))
     (stroke (width 0) (type default))
@@
     (stroke (width 0) (type default))
   )
-  (wire (pts (xy 149.225 107.315) (xy 161.29 107.315))
-    (stroke (width 0) (type default))
-  )
   (wire (pts (xy 335.915 141.605) (xy 335.915 91.44))
     (stroke (width 0) (type default))
   )
-  (wire (pts (xy 134.62 101.6) (xy 161.29 101.6))
-    (stroke (width 0) (type default))
-  )
   (wire (pts (xy 116.84 93.345) (xy 161.29 93.345))
     (stroke (width 0) (type default))
@@
     (stroke (width 0) (type default))
   )
-  (wire (pts (xy 132.08 99.695) (xy 132.08 133.35))
-    (stroke (width 0) (type default))
-  )
   (wire (pts (xy 250.19 111.125) (xy 250.19 142.875))
     (stroke (width 0) (type default))
@@
     (stroke (width 0) (type default))
   )
-  (wire (pts (xy 116.84 135.255) (xy 134.62 135.255))
-    (stroke (width 0) (type default))
-  )
   (wire (pts (xy 332.105 89.535) (xy 337.82 89.535))
     (stroke (width 0) (type default))
   )
-  (symbol (lib_id "Mechanical:Fiducial") (at 335.28 228.6 0) (unit 1)
-    (in_bom yes) (on_board yes) (dnp no) (fields_autoplaced)
-    (property "Reference" "FID1" (at 337.439 227.6915 0)
-      (effects (font (size 1.27 1.27)) (justify left))
-    )
-    (property "Value" "Fiducial" (at 337.439 230.4666 0)
-      (effects (font (size 1.27 1.27)) (justify left))
-    )
-    (property "Footprint" "personal:Product Stamp" (at 335.28 228.6 0)
-      (effects (font (size 1.27 1.27)) hide)
-    )
-    (property "Datasheet" "~" (at 335.28 228.6 0)
-      (effects (font (size 1.27 1.27)) hide)
-    )
-    (instances
-      (project "Grower"
-        (path "/1fa508ef-df83-4c99-846b-9acf535b3ad9"
-          (reference "FID1") (unit 1)
-        )
-      )
-    )
-  )
   (sheet (at 274.32 124.46) (size 57.15 40.005) (fields_autoplaced)
     (stroke (width 0.1524) (type solid))
@@
     )
     (instances
-      (project "Grower"
+      (project "PlantBot"
         (path "/1fa508ef-df83-4c99-846b-9acf535b3ad9" (page "5"))
       )
@@
     )
     (instances
-      (project "Grower"
+      (project "PlantBot"
         (path "/1fa508ef-df83-4c99-846b-9acf535b3ad9" (page "3"))
       )
@@
     )
     (instances
-      (project "Grower"
+      (project "PlantBot"
         (path "/1fa508ef-df83-4c99-846b-9acf535b3ad9" (page "4"))
       )
@@
     )
     (instances
-      (project "Grower"
+      (project "PlantBot"
         (path "/1fa508ef-df83-4c99-846b-9acf535b3ad9" (page "2"))
       )
@@
       (effects (font (size 1.27 1.27)) (justify left))
     )
-    (pin "SDA" input (at 161.29 99.695 180)
-      (effects (font (size 1.27 1.27)) (justify left))
-    )
-    (pin "SCL" input (at 161.29 101.6 180)
-      (effects (font (size 1.27 1.27)) (justify left))
-    )
     (pin "IN2" input (at 214.63 111.125 0)
       (effects (font (size 1.27 1.27)) (justify right))
@@
       (effects (font (size 1.27 1.27)) (justify right))
     )
-    (pin "STH20_PWR" input (at 161.29 97.79 180)
-      (effects (font (size 1.27 1.27)) (justify left))
-    )
-    (pin "LIGHT_MIC_PWR" input (at 161.29 105.41 180)
-      (effects (font (size 1.27 1.27)) (justify left))
-    )
     (pin "LIGHT_SIG" input (at 161.29 109.22 180)
       (effects (font (size 1.27 1.27)) (justify left))
     )
-    (pin "AMP_MIC_OUT" input (at 161.29 107.315 180)
-      (effects (font (size 1.27 1.27)) (justify left))
-    )
     (pin "USB_DN" input (at 214.63 84.455 0)
       (effects (font (size 1.27 1.27)) (justify right))
@@
       (effects (font (size 1.27 1.27)) (justify right))
     )
-    (instances
-      (project "Grower"
+    (pin "LIGHT_PWR" input (at 161.29 107.315 180)
+      (effects (font (size 1.27 1.27)) (justify left))
+    )
+    (instances
+      (project "PlantBot"
         (path "/1fa508ef-df83-4c99-846b-9acf535b3ad9" (page "6"))
       )
@@
       (effects (font (size 1.27 1.27)) (justify left top))
     )
-    (pin "SCL" input (at 116.84 133.35 0)
-      (effects (font (size 1.27 1.27)) (justify right))
-    )
-    (pin "SDA" input (at 116.84 135.255 0)
-      (effects (font (size 1.27 1.27)) (justify right))
-    )
-    (pin "SHT20_PWR" input (at 116.84 131.445 0)
-      (effects (font (size 1.27 1.27)) (justify right))
-    )
-    (pin "AMP_MIC_OUT" input (at 116.84 151.13 0)
-      (effects (font (size 1.27 1.27)) (justify right))
-    )
     (pin "LIGHT_SIG" input (at 116.84 153.035 0)
       (effects (font (size 1.27 1.27)) (justify right))
     )
-    (pin "LIGHT_MIC_PWR" input (at 116.84 147.955 0)
-      (effects (font (size 1.27 1.27)) (justify right))
-    )
-    (instances
-      (project "Grower"
+    (pin "LIGHT_PWR" input (at 116.84 151.13 0)
+      (effects (font (size 1.27 1.27)) (justify right))
+    )
+    (instances
+      (project "PlantBot"
         (path "/1fa508ef-df83-4c99-846b-9acf535b3ad9" (page "9"))
       )

Commit message: Completed initial schematic
Parts:
- added C1: 10u, Capacitor_SMD:C_0805_2012Metric, symbol Capacitor_JLC:10u
- added D2: Green_0603, LED_SMD:LED_0603_1608Metric, symbol Diode_JLC:Green_0603
- added J1: GT-USB-7010, Connectors_JT:GT-USB-7010A, symbol Connector_JLC:GT-USB-7010
- added J2: SM04B-SRSS-TB__LF__SN_, SM04BSRSSTBLFSN, symbol Connector_JLC:SM04B-SRSS-TB__LF__SN_
- added J3: KF350-3.5-2P, KF350352P, symbol Connector_JLC:KF350-3.5-2P
- added JP2: Jumper_2_Open, Jumper:SolderJumper-2_P1.3mm_Open_RoundedPad1.0x1.5mm, symbol Jumper:Jumper_2_Open
- added Q1: BSS138, Package_TO_SOT_SMD:SOT-23, symbol Transistor_JLC:BSS138
- added R1, R2: 5.1k, Resistor_SMD:R_0402_1005Metric, symbol Resistor_JLC:5.1k
- added R15: 220, Resistor_SMD:R_0402_1005Metric, symbol Resistor_JLC:220
- added R7: 2.2k, Resistor_SMD:R_0402_1005Metric, symbol Resistor_JLC:2.2k
- added TP1, TP2, TP3: TestPoint_Alt, TestPoint:TestPoint_Pad_1.0x1.0mm, symbol personal:TestPoint_Alt
Connections:
- new net: D2.2 (A), R7.1
- new net: J1.A5 (CC1), R2.1
- new net: J3.2, JP2.1 (A), Q1.3 (D)
- new net: J1.B5 (CC2), R1.1
- new net: Q1.1 (G), R15.2
- new net +3V3: J2.2, TP3.1
- new net Battery Charger/VUSB: C1.2, J1.A4 (VBUS), J1.A9 (VBUS), J1.B4 (VBUS), J1.B9 (VBUS), R7.2
- new net GND: C1.1, D2.1 (K), J1.A1 (GND), J1.B1 (GND), J1.S1 (SHIELD), J2.1, JP2.2 (B), Q1.2 (S), R1.2, R2.2, TP1.1
- new net MCU_DM: J1.A7 (D-), J1.B7 (D-)
- new net MCU_DP: J1.A6 (D+), J1.B6 (D+)
- new net Microcontroller/I2C_SCL: J2.4
- new net Microcontroller/I2C_SDA: J2.3
- new net Microcontroller/PUMP_DRIVE: R15.1
- new net VDD: J3.1, TP2.1
- no-connect marks 0 -> 4
Other:
- removed sheet Capacitive Moisture Sensor
- removed sheet Connectors
- removed sheet Pump Driver
- added sheet Battery Charger (charger.kicad_sch)
- sheet Microcontroller ports: added BAT, CAP_SIG, I2C_SCL, I2C_SDA, PUMP_DRIVE, READ_BATT, USB_DM; removed IN1, IN2, SIG, USB_DN
- sheet Power ports: added 3V3, VDD; removed none
- sheet Sensor ports: added CAP_SIG, I2C_SCL, I2C_SDA; removed none
- note added: "PUMP"
- note added: "QWIIC"

Commit message: updated design
Parts:
- removed J3: KF350-3.5-2P, KF350352P, symbol Connector_JLC:KF350-3.5-2P
- removed JP2: Jumper_2_Open, Jumper:SolderJumper-2_P1.3mm_Open_RoundedPad1.0x1.5mm, symbol Jumper:Jumper_2_Open
- added C20: 1u, Capacitor_SMD:C_0402_1005Metric, symbol Capacitor_JLC:1u
- added D5: 1N4148WS, Diode_SMD:D_SOD-323F, symbol Diode_JLC:1N4148WS
- added J4: 2060-452_998-404, 2060452998404, symbol Connector_JLC:2060-452_998-404
- added R17, R18: 10k, Resistor_SMD:R_0402_1005Metric, symbol Resistor_JLC:10k
Connections:
- net GND: now also C20.2, D5.2 (A)
- net Microcontroller/I2C_SCL: now also R18.2
- net Microcontroller/I2C_SDA: now also R17.2
- net Microcontroller/LIGHT_PWR: now also R17.1, R18.1
- net VDD: now also C20.1, J4.1 (1.1), J4.2 (1.2)
- net at Q1.3 (D): now also D5.1 (K), J4.3 (2.1), J4.4 (2.2)
Other:
- moved on the sheet: Q1

Commit message: created fab files
Parts:
- removed C1: 10u, Capacitor_SMD:C_0805_2012Metric, symbol Capacitor_JLC:10u
- removed C20: 1u, Capacitor_SMD:C_0402_1005Metric, symbol Capacitor_JLC:1u
- removed D2: Green_0603, LED_SMD:LED_0603_1608Metric, symbol Diode_JLC:Green_0603
- removed D5: 1N4148WS, Diode_SMD:D_SOD-323F, symbol Diode_JLC:1N4148WS
- removed J4: 2060-452_998-404, 2060452998404, symbol Connector_JLC:2060-452_998-404
- removed Q1: BSS138, Package_TO_SOT_SMD:SOT-23, symbol Transistor_JLC:BSS138
- removed R15: 220, Resistor_SMD:R_0402_1005Metric, symbol Resistor_JLC:220
- removed R7: 2.2k, Resistor_SMD:R_0402_1005Metric, symbol Resistor_JLC:2.2k
Other:
- added sheet Pump (pump.kicad_sch)
- note removed: "PUMP"

Commit message: updated prod files with fiducials
Parts:
- added FID1: Fiducial, personal:Product Stamp, symbol Mechanical:Fiducial
- added FID2: Fiducial, personal:jlcpcb_logo_2mm, symbol Mechanical:Fiducial
Changed lines of the file:
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@@
 	(title_block
 		(title "Plant Bot")
-		(date "2025-01-13")
+		(date "2025-01-22")
 		(rev "F")
 	)
@@
 				(path "/1fa508ef-df83-4c99-846b-9acf535b3ad9"
 					(reference "R17")
+					(unit 1)
+				)
+			)
+		)
+	)
+	(symbol
+		(lib_id "Mechanical:Fiducial")
+		(at 280.162 245.364 0)
+		(unit 1)
+		(exclude_from_sim yes)
+		(in_bom no)
+		(on_board yes)
+		(dnp no)
+		(fields_autoplaced yes)
+		(property "Reference" "FID2"
+			(at 282.321 244.1518 0)
+			(effects
+				(font
+					(size 1.27 1.27)
+				)
+				(justify left)
+			)
+		)
+		(property "Value" "Fiducial"
+			(at 282.321 246.5761 0)
+			(effects
+				(font
+					(size 1.27 1.27)
+				)
+				(justify left)
+			)
+		)
+		(property "Footprint" "personal:jlcpcb_logo_2mm"
+			(at 280.162 245.364 0)
+			(effects
+				(font
+					(size 1.27 1.27)
+				)
+				(hide yes)
+			)
+		)
+		(property "Datasheet" "~"
+			(at 280.162 245.364 0)
+			(effects
+				(font
+					(size 1.27 1.27)
+				)
+				(hide yes)
+			)
+		)
+		(property "Description" "Fiducial Marker"
+			(at 280.162 245.364 0)
+			(effects
+				(font
+					(size 1.27 1.27)
+				)
+				(hide yes)
+			)
+		)
+		(instances
+			(project ""
+				(path "/1fa508ef-df83-4c99-846b-9acf535b3ad9"
+					(reference "FID2")
 					(unit 1)
 				)
@@
 					(unit 1)
 				)
+			)
+		)
+	)
+	(symbol
+		(lib_id "Mechanical:Fiducial")
+		(at 280.416 238.76 0)
+		(unit 1)
+		(exclude_from_sim yes)
+		(in_bom no)
+		(on_board yes)
+		(dnp no)
+		(fields_autoplaced yes)
+		(property "Reference" "FID1"
+			(at 282.575 237.5478 0)
+			(effects
+				(font
+					(size 1.27 1.27)
+				)
+				(justify left)
+			)
+		)
+		(property "Value" "Fiducial"
+			(at 282.575 239.9721 0)
+			(effects
+				(font
+					(size 1.27 1.27)
+				)
+				(justify left)
+			)
+		)
+		(property "Footprint" "personal:Product Stamp"
+			(at 280.416 238.76 0)
+			(effects
+				(font
+					(size 1.27 1.27)
+				)
+				(hide yes)
+			)
+		)
+		(property "Datasheet" "~"
+			(at 280.416 238.76 0)
+			(effects
+				(font
+					(size 1.27 1.27)
+				)
+				(hide yes)
+			)
+		)
+		(property "Description" "Fiducial Marker"
+			(at 280.416 238.76 0)
+			(effects
+				(font
+					(size 1.27 1.27)
+				)
+				(hide yes)
+			)
+		)
+		(instances
+			(project ""
+				(path "/1fa508ef-df83-4c99-846b-9acf535b3ad9"
+					(reference "FID1")
+					(unit 1)
+				)
