File: pcb/charger.kicad_sch (KiCad schematic)
At the start: 20 parts, among them IC6 BQ24073RGTR, U2 CR2032-BS-6-1

Commit message: updated design
Parts:
- removed S3: K3-1296S-E1, K31296SE1, symbol Switches_JLC:K3-1296S-E1
Connections:
- net VDD: now also C18.1, IC6.10 (OUT_1), IC6.11 (OUT_2), R30.2, R31.1, R33.1
- no-connect marks 5 -> 0
Changed lines of the file:
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@@
 	(title_block
 		(title "Plant Bot")
-		(date "2025-01-11")
+		(date "2025-01-13")
 		(rev "F")
 	)
@@
 	)
 	(junction
-		(at 176.276 137.922)
-		(diameter 0)
-		(color 0 0 0 0)
-	)
-	(junction
 		(at 123.571 150.622)
 		(diameter 0)
@@
 	)
 	(junction
+		(at 176.276 137.922)
+		(diameter 0)
+		(color 0 0 0 0)
+	)
+	(junction
 		(at 166.751 137.922)
 		(diameter 0)
@@
 		(color 0 0 0 0)
 	)
-	(no_connect
-		(at 202.946 139.827)
-	)
-	(no_connect
-		(at 202.946 142.367)
-	)
-	(no_connect
-		(at 202.946 137.287)
-	)
-	(no_connect
-		(at 202.946 144.907)
-	)
-	(no_connect
-		(at 201.676 133.477)
-	)
 	(wire
 		(pts
@@
 	(wire
 		(pts
-			(xy 201.676 128.397) (xy 206.756 128.397)
-		)
-		(stroke
-			(width 0)
-			(type default)
-		)
-	)
-	(wire
-		(pts
 			(xy 101.981 179.197) (xy 111.506 179.197)
 		)
@@
 	(wire
 		(pts
-			(xy 176.276 130.937) (xy 176.276 137.922)
-		)
-		(stroke
-			(width 0)
-			(type default)
-		)
-	)
-	(wire
-		(pts
 			(xy 300.736 110.617) (xy 307.721 110.617)
 		)
@@
 	(wire
 		(pts
+			(xy 191.77 131.064) (xy 176.276 131.064)
+		)
+		(stroke
+			(width 0)
+			(type default)
+		)
+	)
+	(wire
+		(pts
 			(xy 160.401 148.082) (xy 166.751 148.082)
 		)
@@
 	(wire
 		(pts
+			(xy 176.276 131.064) (xy 176.276 137.922)
+		)
+		(stroke
+			(width 0)
+			(type default)
+		)
+	)
+	(wire
+		(pts
 			(xy 129.921 163.322) (xy 111.506 163.322)
 		)
@@
 		(pts
 			(xy 119.761 165.862) (xy 119.761 167.132)
-		)
-		(stroke
-			(width 0)
-			(type default)
-		)
-	)
-	(wire
-		(pts
-			(xy 186.436 130.937) (xy 176.276 130.937)
 		)
 		(stroke
@@
 	(hierarchical_label "VDD"
 		(shape input)
-		(at 206.756 128.397 0)
+		(at 191.77 131.064 0)
 		(fields_autoplaced yes)
 		(effects
@@
 					(unit 1)
 				)
-			)
-		)
-	)
-	(symbol
-		(lib_id "Switches_JLC:K3-1296S-E1")
-		(at 185.166 123.317 0)
-		(unit 1)
-		(exclude_from_sim no)
-		(in_bom yes)
-		(on_board yes)
-		(dnp no)
-		(fields_autoplaced yes)
-		(property "Reference" "S3"
-			(at 194.056 122.0175 0)
-			(effects
-				(font
-					(size 1.27 1.27)
-				)
-			)
-		)
-		(property "Value" "K3-1296S-E1"
-			(at 194.056 124.7926 0)
-			(effects
-				(font
-					(size 1.27 1.27)
-				)
-			)
-		)
-		(property "Footprint" "K31296SE1"
-			(at 206.756 120.777 0)
-			(effects
-				(font
-					(size 1.27 1.27)
-				)
-				(justify left)
-				(hide yes)
-			)
-		)
-		(property "Datasheet" "https://datasheet.lcsc.com/szlcsc/Korean-Hroparts-Elec-K3-1296S-E1_C128955.pdf"
-			(at 206.756 123.317 0)
-			(effects
-				(font
-					(size 1.27 1.27)
-				)
-				(justify left)
-				(hide yes)
-			)
-		)
-		(property "Description" "Toggle Switches SMD RoHS"
-			(at 206.756 125.857 0)
-			(effects
-				(font
-					(size 1.27 1.27)
-				)
-				(justify left)
-				(hide yes)
-			)
-		)
-		(property "Height" "1.6"
-			(at 206.756 128.397 0)
-			(effects
-				(font
-					(size 1.27 1.27)
-				)
-				(justify left)
-				(hide yes)
-			)
-		)
-		(property "Manufacturer_Name" "Korean Hroparts Elec"
-			(at 206.756 130.937 0)
-			(effects
-				(font
-					(size 1.27 1.27)
-				)
-				(justify left)
-				(hide yes)
-			)
-		)
-		(property "Manufacturer_Part_Number" "K3-1296S-E1"
-			(at 202.946 114.427 0)
-			(effects
-				(font
-					(size 1.27 1.27)
-				)
-				(justify left)
-				(hide yes)
-			)
-		)
-		(property "LCSC" "C128955"
-			(at 185.166 123.317 0)
-			(effects
-				(font
-					(size 1.27 1.27)
-				)
-				(hide yes)
-			)
-		)
-		(pin "MP1"
-		)
-		(pin "MP2"
-		)
-		(pin "MP3"
-		)
-		(pin "MP4"
-		)
-		(pin "1"
-		)
-		(pin "2"
-		)
-		(pin "3"
-		)
-		(instances
-			(project "PlantBot"
-				(path "/1fa508ef-df83-4c99-846b-9acf535b3ad9/64bb1079-49be-4a7d-93cf-555cc5d3e35c"
-					(reference "S3")
-					(unit 1)
-				)
