File: pcb/microcontroller.kicad_sch (KiCad schematic)
At the start: 17 parts, among them IC5 ESP32-C3-MINI-1-N4, Q1 MUN5214DW1T1G

Commit message: created step file
Parts:
- removed Q1: MUN5214DW1T1G, Package_TO_SOT_SMD:SOT-363_SC-70-6, symbol Transistor_JLC:MUN5214DW1T1G
- removed TP12 (x2): TestPoint_Alt, TestPoint:TestPoint_Pad_1.0x1.0mm, symbol personal:TestPoint_Alt
Connections:
- net AMP_MIC_OUT: no longer names the net of IC5.13 (IO1)
- net LIGHT_MIC_PWR renamed LIGHT_PWR
- net STH20_PWR: no longer names the net of IC5.6 (IO3)
- net U0RXD: no longer names the net of IC5.30 (RXD0)
- net U0TXD: no longer names the net of IC5.31 (TXD0)
- no-connect marks 15 -> 19
Other:
- note removed: "AUTO PROGRAM"

Commit message: Completed initial schematic
Parts:
- removed C14: 1u, Capacitor_SMD:C_0402_1005Metric, symbol Capacitor_JLC:1u
- removed C15, C19, C20: 100n, Capacitor_SMD:C_0402_1005Metric, symbol Capacitor_JLC:100n
- removed C16: 10u, Capacitor_SMD:C_0805_2012Metric, symbol Capacitor_JLC:10u
- removed IC5: ESP32-C3-MINI-1-N4, ESP32C3MINI1N4, symbol MCU_JLC:ESP32-C3-MINI-1-N4
- removed LED1: WS2812B-4020, WS2812B4020, symbol Diode_JLC:WS2812B-4020
- removed R10, R11, R22: 10k, Resistor_SMD:R_0402_1005Metric, symbol Resistor_JLC:10k
- added C10, C11, C8: 100n, Capacitor_SMD:C_0402_1005Metric, symbol Capacitor_JLC:100n
- added C7: 10u, Capacitor_SMD:C_0805_2012Metric, symbol Capacitor_JLC:10u
- added C9: 1u, Capacitor_SMD:C_0402_1005Metric, symbol Capacitor_JLC:1u
- added D3: Red_0603, LED_SMD:LED_0603_1608Metric, symbol Diode_JLC:Red_0603
- added D7: Yellow_0603, LED_SMD:LED_0603_1608Metric, symbol Diode_JLC:Yellow_0603
- added D8: Green_0603, LED_SMD:LED_0603_1608Metric, symbol Diode_JLC:Green_0603
- added IC3: ESP32-C6-MINI-1-N4, ESP32C6MINI1N4, symbol MCU_JLC:ESP32-C6-MINI-1-N4
- added JP1: Jumper_2_Bridged, Jumper:SolderJumper-2_P1.3mm_Bridged_RoundedPad1.0x1.5mm, symbol Jumper:Jumper_2_Bridged
- added R10, R11, R12: 330, Resistor_SMD:R_0402_1005Metric, symbol Resistor_JLC:330
- added R14, R8: 10k, Resistor_SMD:R_0402_1005Metric, symbol Resistor_JLC:10k
Connections:
- net +3V3: now also JP1.1 (A), R14.1
- net CHIP_PU: now also C11.2, C9.2, IC3.8 (EN), R8.1
- net GND: now also C10.1, C11.1, C7.2, C8.2, C9.1, IC3.1 (GND_1), IC3.11 (GND_3), IC3.14 (GND_4), IC3.2 (GND_2), IC3.36 (GND_5), IC3.37 (GND_6), IC3.38 (GND_7), IC3.39 (GND_8), IC3.40 (GND_9), IC3.41 (GND_10), IC3.42 (GND_11), IC3.43 (GND_12), IC3.44 (GND_13), IC3.45 (GND_14), IC3.46 (GND_15), IC3.47 (GND_16), IC3.48 (GND_17), IC3.49 (GND_18), IC3.50 (GND_19), IC3.51 (GND_20), IC3.52 (GND_21), IC3.53 (GND_22), IC3.54 (GND_23), IC3.55 (GND_24), IC3.56 (GND_25), IC3.57 (GND_26), IC3.58 (GND_27), IC3.59 (GND_28), IC3.60 (GND_29), IC3.61 (GND_30), R10.2, R11.2, R12.2
- net GPIO8: now also IC3.22 (IO8), R14.2
- net GPIO9: now also C10.2, IC3.23 (IO9)
- net LIGHT_PWR: now also IC3.6 (IO3)
- net LIGHT_SIG: now also IC3.5 (IO2)
- net USB_DP: now also IC3.18 (IO13)
- net at D4.1 (K): now also R11.1; no longer R13.1
- net IND_LED: no longer names the net of D4.2 (A)
- net IND_LED: now also IC3.28 (IO22)
- new net: C7.1, C8.1, IC3.3 (3V3), JP1.2 (B), R8.2
- new net: D7.1 (K), R12.1
- new net: D7.2 (A), IC3.27 (IO21)
- new net: D3.1 (K), R10.1
- new net: D3.2 (A), IC3.29 (IO23)
- new net: D8.1 (K), R13.1
- new net CAP_SIG: IC3.9 (IO4)
- new net DB_LED: D8.2 (A), IC3.12 (IO0)
- new net I2C_SCL: IC3.20 (IO15)
- new net I2C_SDA: IC3.19 (IO14)
- new net PUMP_DRIVE: IC3.10 (IO5)
- new net READ_BATT: IC3.13 (IO1)
- new net USB_DM: IC3.17 (IO12)
- no-connect marks 19 -> 14
Other:
- note added: "READ_BATT and DEBUG_LED are same pins."
- note removed: "ADC1_CH0"
- note removed: "ADC1_CH1"

Commit message: updated design
Parts:
- removed D3: Red_0603, LED_SMD:LED_0603_1608Metric, symbol Diode_JLC:Red_0603
- removed D4: Green_0603, LED_SMD:LED_0603_1608Metric, symbol Diode_JLC:Green_0603
- removed D7: Yellow_0603, LED_SMD:LED_0603_1608Metric, symbol Diode_JLC:Yellow_0603
- removed R10, R11, R12: 330, Resistor_SMD:R_0402_1005Metric, symbol Resistor_JLC:330
Connections:
- no-connect marks 14 -> 17

Commit message: created fab files
Parts:
- removed JP1: Jumper_2_Bridged, Jumper:SolderJumper-2_P1.3mm_Bridged_RoundedPad1.0x1.5mm, symbol Jumper:Jumper_2_Bridged
Connections:
- net +3V3: now also C7.1, C8.1, IC3.3 (3V3), R8.2
- net BAT: now reaches IC3.15 (IO6)
- no-connect marks 17 -> 16
Changed lines of the file:
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@@
-	)
-	(junction
-		(at 101.6 127.508)
-		(diameter 0)
-		(color 0 0 0 0)
 	)
 	(junction
@@
 	)
 	(junction
+		(at 61.595 111.7026)
+		(diameter 0)
+		(color 0 0 0 0)
+	)
+	(junction
 		(at 147.32 178.308)
 		(diameter 0)
@@
 	)
 	(no_connect
-		(at 114.3 142.748)
-	)
-	(no_connect
 		(at 217.805 145.288)
 	)
@@
 	(wire
 		(pts
-			(xy 101.6 127.508) (xy 114.3 127.508)
-		)
-		(stroke
-			(width 0)
-			(type default)
-		)
-	)
-	(wire
-		(pts
 			(xy 86.36 124.968) (xy 86.36 127.508)
 		)
@@
 	(wire
 		(pts
+			(xy 61.595 111.7026) (xy 61.595 117.348)
+		)
+		(stroke
+			(width 0)
+			(type default)
+		)
+	)
+	(wire
+		(pts
 			(xy 193.04 178.308) (xy 195.58 178.308)
 		)
@@
 	(wire
 		(pts
-			(xy 61.595 111.633) (xy 61.595 117.348)
-		)
-		(stroke
-			(width 0)
-			(type default)
-		)
-	)
-	(wire
-		(pts
-			(xy 101.6 130.048) (xy 101.6 127.508)
+			(xy 61.595 111.633) (xy 61.595 111.7026)
 		)
 		(stroke
@@
 	(wire
 		(pts
+			(xy 42.926 111.7026) (xy 42.926 101.6)
+		)
+		(stroke
+			(width 0)
+			(type default)
+		)
+	)
+	(wire
+		(pts
 			(xy 195.58 178.308) (xy 198.12 178.308)
 		)
@@
 	(wire
 		(pts
-			(xy 94.615 130.048) (xy 101.6 130.048)
-		)
-		(stroke
-			(width 0)
-			(type default)
-		)
-	)
-	(wire
-		(pts
 			(xy 73.66 117.348) (xy 73.66 119.253)
 		)
@@
 	(wire
 		(pts
+			(xy 61.595 111.7026) (xy 42.926 111.7026)
+		)
+		(stroke
+			(width 0)
+			(type default)
+		)
+	)
+	(wire
+		(pts
 			(xy 137.16 178.308) (xy 139.7 178.308)
 		)
@@
 	(wire
 		(pts
-			(xy 42.545 100.838) (xy 42.545 111.633)
-		)
-		(stroke
-			(width 0)
-			(type default)
-		)
-	)
-	(wire
-		(pts
 			(xy 104.14 121.158) (xy 107.315 121.158)
 		)
@@
 	(wire
 		(pts
-			(xy 59.055 111.633) (xy 61.595 111.633)
-		)
-		(stroke
-			(width 0)
-			(type default)
-		)
-	)
-	(wire
-		(pts
 			(xy 182.88 178.308) (xy 185.42 178.308)
 		)
@@
 	(wire
 		(pts
-			(xy 99.06 127.508) (xy 101.6 127.508)
+			(xy 99.06 127.508) (xy 114.3 127.508)
 		)
 		(stroke
@@
 		(pts
 			(xy 124.46 178.308) (xy 127 178.308)
-		)
-		(stroke
-			(width 0)
-			(type default)
-		)
-	)
-	(wire
-		(pts
-			(xy 42.545 111.633) (xy 48.895 111.633)
 		)
 		(stroke
@@
 	(hierarchical_label "BAT"
 		(shape input)
-		(at 94.615 130.048 180)
+		(at 114.3 142.748 180)
 		(fields_autoplaced yes)
 		(effects
@@
 		(lib_name "+3V3_1")
 		(lib_id "power:+3V3")
-		(at 42.545 100.838 0)
+		(at 42.926 101.6 0)
 		(unit 1)
 		(exclude_from_sim no)
@@
 		(fields_autoplaced yes)
 		(property "Reference" "#PWR07"
-			(at 42.545 104.648 0)
+			(at 42.926 105.41 0)
 			(effects
 				(font
@@
 		)
 		(property "Value" "+3V3"
-			(at 42.545 97.3361 0)
+			(at 42.926 98.0981 0)
 			(effects
 				(font
@@
 		)
 		(property "Footprint" ""
-			(at 42.545 100.838 0)
+			(at 42.926 101.6 0)
 			(effects
 				(font
@@
 		)
 		(property "Datasheet" ""
-			(at 42.545 100.838 0)
+			(at 42.926 101.6 0)
 			(effects
 				(font
@@
 		)
 		(property "Description" ""
-			(at 42.545 100.838 0)
+			(at 42.926 101.6 0)
 			(effects
 				(font
@@
 					(unit 1)
 				)
-			)
-		)
-	)
-	(symbol
-		(lib_id "Jumper:Jumper_2_Bridged")
-		(at 53.975 111.633 0)
-		(unit 1)
-		(exclude_from_sim no)
-		(in_bom yes)
-		(on_board yes)
-		(dnp no)
-		(fields_autoplaced yes)
-		(property "Reference" "JP1"
-			(at 53.975 107.9881 0)
-			(effects
-				(font
-					(size 1.27 1.27)
-				)
-			)
-		)
-		(property "Value" "Jumper_2_Bridged"
-			(at 53.975 109.9091 0)
-			(effects
-				(font
-					(size 1.27 1.27)
-				)
-			)
-		)
-		(property "Footprint" "Jumper:SolderJumper-2_P1.3mm_Bridged_RoundedPad1.0x1.5mm"
-			(at 53.975 111.633 0)
-			(effects
-				(font
-					(size 1.27 1.27)
-				)
-				(hide yes)
-			)
-		)
-		(property "Datasheet" "~"
-			(at 53.975 111.633 0)
-			(effects
-				(font
-					(size 1.27 1.27)
-				)
-				(hide yes)
-			)
-		)
-		(property "Description" ""
-			(at 53.975 111.633 0)
-			(effects
-				(font
-					(size 1.27 1.27)
-				)
-				(hide yes)
-			)
-		)
-		(pin "1"
-		)
-		(pin "2"
-		)
-		(instances
-			(project "PlantBot"
-				(path "/1fa508ef-df83-4c99-846b-9acf535b3ad9/153a9d0e-b2bb-47fb-80f5-e280eabd2f18"
-					(reference "JP1")
-					(unit 1)
-				)
