File: pcb/plantBot.kicad_pcb (KiCad board)
At the start: 4 copper layers, 36 x 115.4 mm, 92 parts, among them IC1 NE555DR, IC2 LM358DR2G, IC3 XC6227C331MR-G, IC4 DRV8837CDSGR, IC5 ESP32-C3-MINI-1-N4, IC6 BQ24073RGTR, IC7 SHT20, J1 GT-USB-7010, J6 KF350-3.5-2P, Q1 MUN5214DW1T1G, Q2 TEMT6000X01, U1 USBLC6-2P6, U3 CR2032-BS-6-1, U4 LMV321

Commit message: created step file
Parts:
- removed C12, C13: 10u, Capacitor_SMD:C_0805_2012Metric
- removed C21, C28: 100n, Capacitor_SMD:C_0402_1005Metric
- removed C25: 4.7u, Capacitor_SMD:C_1206_3216Metric
- removed C26: 1u, Capacitor_SMD:C_0402_1005Metric
- removed C27: 27p, Capacitor_SMD:C_0402_1005Metric
- removed FID1: Fiducial, personal:Product Stamp
- removed IC7: SHT20, SamacSys_Parts:SON100P300X300X110-7N
- removed MK1: AP2718AT, SamacSys_Parts:AP2718AT
- removed Q1: MUN5214DW1T1G, Package_TO_SOT_SMD:SOT-363_SC-70-6
- removed R27: DNF_0805, Resistor_SMD:R_0805_2012Metric_Pad1.20x1.40mm_HandSolder
- removed R31: 4.7k, Resistor_SMD:R_0402_1005Metric
- removed R32, R33, R7, R8: 10k, Resistor_SMD:R_0402_1005Metric
- removed R34: 300k, Resistor_SMD:R_0402_1005Metric
- removed TP1, TP2: TestPoint_Alt, TestPoint:TestPoint_Pad_1.0x1.0mm
- removed U4: LMV321, Package_TO_SOT_SMD:SOT-23-5
- added ?: LOGO, personal:battery, B.Cu at (204.2, 103.8)
- added C9: 10u_0402, Capacitor_SMD:C_0402_1005Metric, F.Cu at (221.6, 96.6)
- added G***: LOGO, personal:settings, F.Cu at (211.2, 118.3)
- added G***: LOGO, personal:moistureSensor, F.Cu at (218.3, 157.2)
- added G***: LOGO, personal:coinCell, B.Cu at (204.2, 101.8)
- added G***: LOGO, personal:positive, B.Cu at (208.1, 88.0)
- added G***: LOGO, personal:negative, B.Cu at (207.8, 118.1)
- added G***: LOGO, personal:warning, F.Cu at (213.9, 119.3)
- added G***: LOGO, personal:reset, F.Cu at (229.8, 102.5)
- added G***: LOGO, personal:charging, F.Cu at (210.1, 98.7)
- added G***: LOGO, personal:powerGood, F.Cu at (206.4, 105.6)
- added G***: LOGO, personal:lightSensor, F.Cu at (205.8, 117.5)
- added G***: LOGO, personal:pump, F.Cu at (229.8, 95.0)
- added G***: LOGO, personal:USBC, F.Cu at (218.3, 95.0)
- added G***: LOGO, personal:PlantBot, F.Cu at (213.8, 103.8)
- C8: value 100n -> 10u_0402
- R1, R2: value 4.7k -> 5.1k
- moved R35 31.4 mm to (203.0, 113.5), turned to 180 degrees
- moved R1 28.1 mm to (213.2, 94.5), turned to -90 degrees
- moved R2 28.0 mm to (216.3, 94.5), turned to -90 degrees
- moved Q2 27.7 mm to (203.0, 116.5), turned to -90 degrees
- moved C8 24.9 mm to (220.4, 95.7)
- moved D9 12.2 mm to (221.1, 88.5), turned to -90 degrees
- moved D7 12.0 mm to (224.7, 88.3), turned to -90 degrees
- moved R29 11.9 mm to (223.4, 89.8), turned to -90 degrees
- moved R30 9.59 mm to (222.4, 89.9), turned to 90 degrees
- moved IC4 9.58 mm to (219.4, 98.3), turned to -90 degrees
- moved C19 8.95 mm to (215.7, 111.8), turned to 180 degrees
- moved R22 8.55 mm to (210.2, 96.7)
- moved LED1 8.51 mm to (213.8, 98.2)
- moved C11 7.31 mm to (221.2, 98.9), turned to 90 degrees
- moved U1 6.18 mm to (219.1, 101.1)
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Connections:
- net /Microcontroller/LIGHT_MIC_PWR renamed /Microcontroller/LIGHT_PWR
- C8 pad 1: /Microcontroller/STH20_PWR -> VBUS
- IC5 pad 13: /Microcontroller/AMP_MIC_OUT -> unconnected-(IC5-IO1-Pad13)
- IC5 pad 30: /Microcontroller/U0RXD -> unconnected-(IC5-RXD0-Pad30)
- IC5 pad 31: /Microcontroller/U0TXD -> unconnected-(IC5-TXD0-Pad31)
- IC5 pad 6: /Microcontroller/STH20_PWR -> unconnected-(IC5-IO3-Pad6)
- R1 pad 1: +3V3 -> Net-(J1-CC2)
- R1 pad 2: GPIO8 -> GND
- R2 pad 1: +3V3 -> Net-(J1-CC1)
- R2 pad 2: GPIO9 -> GND
Routing:
- net /Microcontroller/LIGHT_PWR: track 60.2 -> 27.9 mm, vias 6 -> 2
- net /Microcontroller/STH20_PWR: track 23.7 -> 0.00 mm, vias 2 -> 0
- net /Microcontroller/AMP_MIC_OUT: track 22.8 -> 0.00 mm, vias 2 -> 0
- net +3V3: track 106.9 -> 87.8 mm
- net /Microcontroller/IN2: track 35.1 -> 17.3 mm
- net /Microcontroller/IN1: track 34.1 -> 17.3 mm
- net GPIO9: track 22.4 -> 9.21 mm
- net /Connectors/USB_DN: track 30.2 -> 19.0 mm
- net Net-(U4-+): track 10.5 -> 0.00 mm
- net /Connectors/USB_DP: track 26.9 -> 17.3 mm
- net CHIP_PU: track 19.9 -> 10.8 mm, vias 2 -> 0
- net WS2812: track 11.4 -> 19.6 mm
- net GPIO8: track 20.8 -> 13.6 mm, vias 3 -> 2
- net D-: track 5.62 -> 12.5 mm
- net +5V: track 15.5 -> 8.64 mm, vias 1 -> 0
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Other:
- board size 36 x 115.4 mm -> 33.7 x 111.6 mm
- board text added: "Designed by elektroThing"
- board text added: "PlantBot"
- board text removed: "CG"
- board text removed: "Capacitive Moisture Sensor"
- board text removed: "PG"
- board text removed: "PUMP"

Commit message: Added demo scripts
Parts:
- removed D2, D3: RedLED, Diode_SMD:D_0805_2012Metric
- removed JP1: SB_NC, Jumper:SolderJumper-2_P1.3mm_Bridged_Pad1.0x1.5mm
- removed R15: 4.7k, Resistor_SMD:R_0402_1005Metric
- removed R17: 2.2k, Resistor_SMD:R_0402_1005Metric
Routing:
- net Net-(JP1-B): track 33.8 -> 0.00 mm, vias 2 -> 0
- net Net-(D3-K): track 6.00 -> 0.00 mm
- net Net-(D2-K): track 1.82 -> 0.00 mm
- net /Capacitive Moisture Sensor/SIG: track 13.0 -> 12.4 mm

Commit message: Completed initial schematic
Parts:
- removed C19, C20, C22: 100n, Capacitor_SMD:C_0402_1005Metric
- removed D5, D6: Green_0603, LED_SMD:LED_0603_1608Metric
- removed J6: KF350-3.5-2P, SamacSys_Parts:KF350352P
- removed LED1: WS2812B-4020, SamacSys_Parts:WS2812B4020
- removed R18: 1.5k, Resistor_SMD:R_0402_1005Metric
- removed R20, R21: 2.2k, Resistor_SMD:R_0402_1005Metric
- removed R23, R24, R25, R26: 10k, Resistor_SMD:R_0402_1005Metric
- removed TH1: 10k_NTC, Resistor_SMD:R_0402_1005Metric
- removed TP12: TestPoint_Alt, TestPoint:TestPoint_Pad_1.0x1.0mm
- removed U1: USBLC6-2P6, Package_TO_SOT_SMD:SOT-666
- removed U3: CR2032-BS-6-1, SamacSys_Parts:CR2032BS61
- added C12: 100n, Capacitor_SMD:C_0402_1005Metric, F.Cu at (141.8, 150.0)
- added C13: 10u, Capacitor_SMD:C_0805_2012Metric, F.Cu at (171.4, 69.3)
- added D10: Green_0603, LED_SMD:LED_0603_1608Metric, F.Cu at (157.8, 93.1)
- added D11: Green_0603, LED_SMD:LED_0603_1608Metric, F.Cu at (157.8, 95.7)
- added D2: Green_0603, LED_SMD:LED_0603_1608Metric, F.Cu at (155.2, 135.6)
- added D3: Red_0603, LED_SMD:LED_0603_1608Metric, F.Cu at (161.2, 144.2)
- added J2: SM04B-SRSS-TB__LF__SN_, SamacSys_Parts:SM04BSRSSTBLFSN, F.Cu at (145.3, 130.4)
- added J3: KF350-3.5-2P, SamacSys_Parts:KF350352P, F.Cu at (143.5, 139.2)
- added JP1: Jumper_2_Bridged, Jumper:SolderJumper-2_P1.3mm_Bridged_RoundedPad1.0x1.5mm, F.Cu at (161.4, 141.1)
- added JP2: Jumper_2_Open, Jumper:SolderJumper-2_P1.3mm_Open_RoundedPad1.0x1.5mm, F.Cu at (152.5, 132.1)
- added L1: 1.5uH, Inductor_SMD:L_0805_2012Metric, F.Cu at (175.9, 74.0)
- added Q1: BSS138, Package_TO_SOT_SMD:SOT-23, F.Cu at (152.7, 128.1)
- added R15: 220, Resistor_SMD:R_0402_1005Metric, F.Cu at (154.6, 139.9)
- added R31: 2.2k, Resistor_SMD:R_0402_1005Metric, F.Cu at (157.2, 76.8)
- added R32: 51k, Resistor_SMD:R_0402_1005Metric, F.Cu at (157.2, 78.8)
- added R33: 51k, Resistor_SMD:R_0402_1005Metric, F.Cu at (160.1, 68.8)
- added R34: 51k, Resistor_SMD:R_0402_1005Metric, F.Cu at (160.1, 70.8)
- added R36: 51k, Resistor_SMD:R_0402_1005Metric, F.Cu at (160.1, 72.8)
- added R37: 560k, Resistor_SMD:R_0603_1608Metric, F.Cu at (157.7, 98.2)
- added R38: 220k, Resistor_SMD:R_0402_1005Metric, F.Cu at (160.1, 74.8)
- added R7: 2.2k, Resistor_SMD:R_0402_1005Metric, F.Cu at (154.6, 137.9)
- added R8: 10k, Resistor_SMD:R_0402_1005Metric, F.Cu at (164.7, 143.9)
- added S3: K3-1296S-E1, SamacSys_Parts:K31296SE1, F.Cu at (161.5, 82.9)
- added TH2: 10k_NTC, Resistor_SMD:R_0402_1005Metric, F.Cu at (160.1, 76.8)
- added TP1: TestPoint_Alt, TestPoint:TestPoint_Pad_1.0x1.0mm, F.Cu at (151.6, 135.9)
- added TP2: TestPoint_Alt, TestPoint:TestPoint_Pad_1.0x1.0mm, F.Cu at (151.6, 138.9)
- added TP3: TestPoint_Alt, TestPoint:TestPoint_Pad_1.0x1.0mm, F.Cu at (151.6, 142.0)
- added TP4: TestPoint_Alt, TestPoint:TestPoint_Pad_1.0x1.0mm, F.Cu at (141.9, 147.5)
- added U2: CR2032-BS-6-1, SamacSys_Parts:CR2032BS61, F.Cu at (146.2, 85.4)
- C10: value 10u -> 100n; footprint Capacitor_SMD:C_0805_2012Metric -> Capacitor_SMD:C_0402_1005Metric
- C14: value 1u -> 1n
- C15: value 100n -> 10u; footprint Capacitor_SMD:C_0402_1005Metric -> Capacitor_SMD:C_0805_2012Metric
- C5: value 4.7u -> 100n; footprint Capacitor_SMD:C_1206_3216Metric -> Capacitor_SMD:C_0402_1005Metric
- C6: value 100n -> 4.7u; footprint Capacitor_SMD:C_0402_1005Metric -> Capacitor_SMD:C_1206_3216Metric
- C8: value 10u_0402 -> 100n
- C9: value 10u_0402 -> 1u
- D7: value Green_0603 -> Yellow_0603
- D8: value 1N5819HWQ-7-F -> Green_0603; footprint SamacSys_Parts:SOD3716X145N -> LED_SMD:LED_0603_1608Metric
- D9: value Green_0603 -> B5819W.SL; footprint LED_SMD:LED_0603_1608Metric -> SamacSys_Parts:B5819WSL
- IC3: value XC6227C331MR-G -> ESP32-C6-MINI-1-N4; footprint SamacSys_Parts:SOT95P280X130-5N -> SamacSys_Parts:ESP32C6MINI1N4
- IC4: value DRV8837CDSGR -> AHT20; footprint SamacSys_Parts:SON50P200X200X80-9N -> SamacSys_Parts:AHT20
- IC5: value ESP32-C3-MINI-1-N4 -> TPS63051RMWR; footprint SamacSys_Parts:ESP32C3MINI1N4 -> SamacSys_Parts:QFN50P250X250X100-12N-D
- R10, R11: value 10k -> 330
- R12: value 100k -> 330
- R14: value 47.5k -> 10k
- R16: value 1.5k -> 1M
- R22: value 10k -> 51k
- R28: value 0 -> 1.5k; footprint Resistor_SMD:R_0805_2012Metric_Pad1.20x1.40mm_HandSolder -> Resistor_SMD:R_0402_1005Metric
- R29: value 2.2k -> 1.5k
- moved R29 68.4 mm to (157.2, 72.8), turned to 0 degrees
- moved R30 67.0 mm to (157.2, 74.8), turned to 0 degrees
- moved IC5 63.0 mm to (176.1, 70.2), turned to 0 degrees
- moved C16 61.9 mm to (171.4, 75.3)
- moved D9 61.8 mm to (159.3, 89.5), turned to 0 degrees
- moved C15 61.3 mm to (171.4, 72.3), turned to 0 degrees
- moved R22 59.9 mm to (157.2, 68.8), turned to 0 degrees
- moved R28 53.6 mm to (157.2, 70.8)
- moved C14 53.0 mm to (175.1, 76.4), turned to 0 degrees
- moved C17 50.3 mm to (157.1, 100.5), turned to 0 degrees
- moved IC3 45.7 mm to (248.1, 90.0)
- moved IC6 12.2 mm to (192.6, 100.0)
Connections:
- net Net-(IC6-BAT_1) renamed +BATT
- C1 pad 1: +5V -> GND
- C1 pad 2: GND -> /Battery Charger/VUSB
- C10 pad 1: +3V3 -> GND
- C10 pad 2: GND -> GPIO9
- C11 pad 1: +3V3 -> GND
- C11 pad 2: GND -> CHIP_PU
- C14 pad 1: CHIP_PU -> Net-(IC5-SS)
- C18 pad 1: VDD -> Net-(IC6-OUT_1)
- C5 pad 1: /Capacitive Moisture Sensor/SIG -> +3V3
- C6 pad 1: +3V3 -> /Microcontroller/CAP_SIG
- C7 pad 1: VDD -> Net-(IC3-3V3)
- C8 pad 1: VBUS -> Net-(IC3-3V3)
- C9 pad 1: VBUS -> GND
- C9 pad 2: GND -> CHIP_PU
- D4 pad 2: IND_LED -> Net-(D4-A)
- D7 pad 1: GND -> Net-(D7-K)
- D8 pad 1: +5V -> Net-(D8-K)
- D8 pad 2: VBUS -> DB_LED
- D9 pad 1: GND -> Net-(IC6-IN)
- D9 pad 2: Net-(D9-A) -> /Battery Charger/VUSB
- IC3 pad 1: VDD -> GND
- IC3 pad 3: Net-(IC3-CE) -> Net-(IC3-3V3)
- IC3 pad 5: +3V3 -> /Microcontroller/LIGHT_SIG
- IC4 pad 1: VBUS -> unconnected-(IC4-NC_1-Pad1)
- IC4 pad 2: /Connectors/OUT_1 -> +3V3
- IC4 pad 3: /Connectors/OUT_2 -> /Microcontroller/I2C_SCL
- IC4 pad 4: GND -> /Microcontroller/I2C_SDA
- IC4 pad 5: /Microcontroller/IN2 -> GND
- IC4 pad 6: /Microcontroller/IN1 -> unconnected-(IC4-NC_2-Pad6)
- IC5 pad 1: GND -> Net-(IC5-L1)
- IC5 pad 10: unconnected-(IC5-NC_4-Pad10) -> VDD
- IC5 pad 11: GND -> VDD
- IC5 pad 12: /Microcontroller/LIGHT_SIG -> VDD
- IC5 pad 3: +3V3 -> Net-(IC5-L2)
- IC5 pad 4: unconnected-(IC5-NC_1-Pad4) -> +3V3
- IC5 pad 5: /Microcontroller/LIGHT_PWR -> +3V3
- IC5 pad 6: unconnected-(IC5-IO3-Pad6) -> GND
- IC5 pad 7: unconnected-(IC5-NC_2-Pad7) -> Net-(IC5-SS)
- IC5 pad 8: CHIP_PU -> Net-(IC5-PG)
- IC5 pad 9: unconnected-(IC5-NC_3-Pad9) -> GND
- IC6 pad 10: VDD -> Net-(IC6-OUT_1)
- IC6 pad 11: VDD -> Net-(IC6-OUT_1)
- J1 pad A4: VBUS -> /Battery Charger/VUSB
- J1 pad A6: D+ -> MCU_DP
- J1 pad A7: D- -> MCU_DM
- J1 pad A9: VBUS -> /Battery Charger/VUSB
- J1 pad B4: VBUS -> /Battery Charger/VUSB
- J1 pad B6: D+ -> MCU_DP
- J1 pad B7: D- -> MCU_DM
- J1 pad B9: VBUS -> /Battery Charger/VUSB
- R10 pad 1: +3V3 -> Net-(D3-K)
- R10 pad 2: CHIP_PU -> GND
- R11 pad 1: +3V3 -> Net-(D4-K)
- R11 pad 2: GPIO8 -> GND
- R12 pad 1: VDD -> Net-(D7-K)
- R12 pad 2: Net-(IC3-CE) -> GND
- R13 pad 1: Net-(D4-K) -> Net-(D8-K)
- R14 pad 1: Net-(IC6-TMR) -> +3V3
- R14 pad 2: GND -> GPIO8
- R16 pad 1: Net-(IC6-ILIM) -> +3V3
- R16 pad 2: GND -> Net-(IC5-PG)
- R22 pad 1: WS2812 -> Net-(IC6-TMR)
- R22 pad 2: +3V3 -> GND
- R28 pad 1: +5V -> Net-(IC6-ILIM)
- R28 pad 2: Net-(IC6-IN) -> GND
- R29 pad 1: Net-(D7-A) -> Net-(IC6-ISET)
- R29 pad 2: /Connectors/OUT_1 -> GND
- R30 pad 1: /Connectors/OUT_2 -> Net-(D10-A)
- R30 pad 2: Net-(D9-A) -> Net-(IC6-OUT_1)
- R9 pad 2: /Capacitive Moisture Sensor/SIG -> /Microcontroller/CAP_SIG
Routing:
- net +3V3: track 87.8 -> 14.8 mm, vias 8 -> 2
- net VBUS: track 31.3 -> 0.00 mm, vias 2 -> 0
- net /Microcontroller/LIGHT_PWR: track 27.7 -> 0.00 mm, vias 2 -> 0
- net VDD: track 26.2 -> 0.00 mm
- net +BATT: track 22.7 -> 0.00 mm, vias 1 -> 0
- net GND: track 144.7 -> 165.9 mm, vias 20 -> 19
- net WS2812: track 19.4 -> 0.00 mm, vias 2 -> 0
- net /Connectors/USB_DN: track 19.0 -> 0.00 mm, vias 2 -> 0
- net /Microcontroller/LIGHT_SIG: track 20.0 -> 2.39 mm
- net /Connectors/USB_DP: track 17.3 -> 0.00 mm, vias 2 -> 0
- net /Microcontroller/IN1: track 17.1 -> 0.00 mm, vias 2 -> 0
- net /Microcontroller/IN2: track 17.1 -> 0.00 mm, vias 2 -> 0
- net /Connectors/OUT_1: track 17.0 -> 0.00 mm
- net /Connectors/OUT_2: track 14.3 -> 0.00 mm
- net D+: track 13.9 -> 0.00 mm
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- removed copper zone on In1.Cu, net GND
- removed copper zone on In2.Cu, net GND
Other:
- copper layers 4 -> 2
- board text added: "| Soil Level |"
- board text removed: "Soil Level"

Commit message: updated design
Parts:
- removed the ? at (204.2, 103.8)
- removed D3: Red_0603, LED_SMD:LED_0603_1608Metric
- removed D4: Green_0603, LED_SMD:LED_0603_1608Metric
- removed D7: Yellow_0603, LED_SMD:LED_0603_1608Metric
- removed G***: LOGO, personal:settings
- removed G***: LOGO, personal:moistureSensor
- removed G***: LOGO, personal:coinCell
- removed G***: LOGO, personal:positive
- removed G***: LOGO, personal:negative
- removed G***: LOGO, personal:warning
- removed G***: LOGO, personal:reset
- removed G***: LOGO, personal:charging
- removed G***: LOGO, personal:powerGood
- removed G***: LOGO, personal:lightSensor
- removed G***: LOGO, personal:pump
- removed G***: LOGO, personal:USBC
- removed G***: LOGO, personal:PlantBot
- removed J3: KF350-3.5-2P, SamacSys_Parts:KF350352P
- removed JP2: Jumper_2_Open, Jumper:SolderJumper-2_P1.3mm_Open_RoundedPad1.0x1.5mm
- removed R10, R11, R12: 330, Resistor_SMD:R_0402_1005Metric
- removed S3: K3-1296S-E1, SamacSys_Parts:K31296SE1
- removed TP4: TestPoint_Alt, TestPoint:TestPoint_Pad_1.0x1.0mm
- added ?: LOGO, personal:PlantBot, B.Cu at (224.5, 89.2)
- added C19: 100n, Capacitor_SMD:C_0402_1005Metric, F.Cu at (205.3, 92.0)
- added C20: 1u, Capacitor_SMD:C_0402_1005Metric, F.Cu at (223.7, 94.1)
- added D5: 1N4148WS, Diode_SMD:D_SOD-323F, F.Cu at (221.1, 94.5)
- added F*: LOGO, personal:logo_10mm, B.Cu at (231.7, 89.2)
- added J4: 2060-452_998-404, SamacSys_Parts:2060452998404, F.Cu at (229.9, 93.1)
- added R17: 10k, Resistor_SMD:R_0402_1005Metric, F.Cu at (207.9, 88.0)
- added R18: 10k, Resistor_SMD:R_0402_1005Metric, F.Cu at (207.9, 89.9)
- added REF**: Product Stamp, personal:Product Stamp, F.Cu at (232.7, 125.8)
- added REF**: OSHW-Logo2_7.3x6mm_SilkScreen, Symbol:OSHW-Logo2_7.3x6mm_SilkScreen, B.Cu at (224.8, 124.8)
- J2, U2: moved to B.Cu
- moved C12 90.0 mm to (227.5, 122.3), turned to 180 degrees
- moved R7 82.2 mm to (222.9, 92.2)
- moved D2 81.5 mm to (222.8, 90.2)
- moved R15 80.8 mm to (223.5, 97.7), turned to -90 degrees
- moved JP1 80.0 mm to (231.8, 103.2), turned to 180 degrees
- moved TP1 78.8 mm to (222.4, 101.2)
- moved Q1 75.0 mm to (221.1, 97.2), turned to 180 degrees
- moved U2 73.9 mm to (218.1, 102.5), turned to -90 degrees
- moved TP3 73.9 mm to (213.3, 101.2)
- moved J2 73.3 mm to (205.5, 88.6)
- moved TP2 70.4 mm to (211.1, 101.2)
- moved R8 69.9 mm to (222.1, 104.2)
- moved R22 66.6 mm to (209.4, 110.2), turned to -90 degrees
- moved R29 66.0 mm to (211.5, 110.2), turned to -90 degrees
- moved R34 63.9 mm to (210.4, 110.2), turned to -90 degrees
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Connections:
- C18 pad 1: Net-(IC6-OUT_1) -> VDD
- IC3 pad 27: Net-(D7-A) -> unconnected-(IC3-IO21-Pad27)
- IC3 pad 28: Net-(D4-A) -> unconnected-(IC3-IO22-Pad28)
- IC3 pad 29: Net-(D3-A) -> unconnected-(IC3-IO23-Pad29)
- IC6 pad 10: Net-(IC6-OUT_1) -> VDD
- IC6 pad 11: Net-(IC6-OUT_1) -> VDD
- R30 pad 2: Net-(IC6-OUT_1) -> VDD
- R31 pad 1: Net-(IC6-OUT_1) -> VDD
- R33 pad 1: Net-(IC6-OUT_1) -> VDD
Routing:
- net +3V3: track 14.8 -> 106.1 mm, vias 2 -> 7
- net VDD: track 0.00 -> 70.4 mm, vias 0 -> 3
- net /Battery Charger/VUSB: track 0.00 -> 41.4 mm, vias 0 -> 5
- net /Microcontroller/LIGHT_PWR: track 0.00 -> 39.5 mm, vias 0 -> 3
- net /Microcontroller/I2C_SDA: track 0.00 -> 38.9 mm, vias 0 -> 2
- net /Microcontroller/I2C_SCL: track 0.00 -> 34.3 mm, vias 0 -> 2
- net CHIP_PU: track 0.00 -> 28.2 mm, vias 0 -> 2
- net GND: track 165.9 -> 139.5 mm, vias 19 -> 33
- net MCU_DP: track 2.58 -> 24.8 mm
- net Net-(D5-K): track 0.00 -> 20.7 mm
- net MCU_DM: track 3.44 -> 23.3 mm
- net /Microcontroller/CAP_SIG: track 0.00 -> 18.4 mm, vias 0 -> 2
- net +BATT: track 0.00 -> 15.6 mm, vias 0 -> 1
- net /Microcontroller/LIGHT_SIG: track 2.39 -> 17.1 mm, vias 0 -> 2
- net GPIO9: track 0.00 -> 13.6 mm
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- added copper zone on F.Cu, net +3V3
- added copper zone on B.Cu, net Net-(IC5-L1)
- added copper zone on F.Cu, net Net-(IC5-L1)
- added copper zone on B.Cu, net Net-(IC5-L2)
- added copper zone on F.Cu, net Net-(IC5-L2)
- added copper zone on F.Cu, net VDD
Other:
- board text added: "+"
- board text added: "-"
- board text added: "AHT20"
- board text added: "GPIO9"
- board text added: "LIGHT SENSOR"
- board text added: "LIR2032"
- board text added: "PUMP"
- board text added: "Plant Bot"
- board text added: "QWIIC"
- board text added: "RESET"
- board text added: "SOIL MOISTURE SENSOR"
- board text added: "USB-C"
- board text added: "VDD"
- board text removed: "5V"
- board text removed: "Designed by elektroThing"
- board text removed: "PlantBot"

Commit message: created fab files
Parts:
- removed C1: 10u, Capacitor_SMD:C_0805_2012Metric
- removed D5: 1N4148WS, Diode_SMD:D_SOD-323F
- removed J4: 2060-452_998-404, SamacSys_Parts:2060452998404
- removed JP1: Jumper_2_Bridged, Jumper:SolderJumper-2_P1.3mm_Bridged_RoundedPad1.0x1.5mm
- removed R15: 220, Resistor_SMD:R_0402_1005Metric
- removed REF**: Product Stamp, personal:Product Stamp
- removed REF**: OSHW-Logo2_7.3x6mm_SilkScreen, Symbol:OSHW-Logo2_7.3x6mm_SilkScreen
- added J3: 2060-452_998-404, SamacSys_Parts:2060452998404, F.Cu at (230.1, 93.0)
- added Q3: DMP3017SFG-7, SamacSys_Parts:DMP3007SFG7, F.Cu at (222.4, 96.9)
- added R10: 220, Resistor_SMD:R_0402_1005Metric, F.Cu at (223.7, 89.4)
- added R11: 10k, Resistor_SMD:R_0402_1005Metric, F.Cu at (218.7, 94.0)
- added R12: 1k, Resistor_SMD:R_0402_1005Metric, F.Cu at (220.9, 92.9)
- Q1: value BSS138 -> DTC143ECA-TP; footprint Package_TO_SOT_SMD:SOT-23 -> SamacSys_Parts:SOT95P237X125-3N
- moved C20 11.4 mm to (232.0, 101.9)
- moved Q1 5.75 mm to (223.2, 91.9), turned to -90 degrees
- moved R7 4.23 mm to (223.4, 88.0), turned to 180 degrees
- moved D2 3.48 mm to (223.0, 86.7)
- moved R2 2.05 mm to (218.5, 95.5), turned to -90 degrees
Connections:
- C12 pad 1: +3V3 -> I2C_PWR
- C19 pad 1: +3V3 -> I2C_PWR
- C20 pad 1: VDD -> Net-(J3-1.1)
- C3 pad 1: +3V3 -> I2C_PWR
- C5 pad 1: +3V3 -> I2C_PWR
- C7 pad 1: Net-(IC3-3V3) -> +3V3
- C8 pad 1: Net-(IC3-3V3) -> +3V3
- IC1 pad 4: +3V3 -> I2C_PWR
- IC1 pad 8: +3V3 -> I2C_PWR
- IC2 pad 8: +3V3 -> I2C_PWR
- IC3 pad 15: unconnected-(IC3-IO6-Pad15) -> /Battery Charger/BAT
- IC3 pad 3: Net-(IC3-3V3) -> +3V3
- IC3 pad 6: /Microcontroller/LIGHT_PWR -> I2C_PWR
- IC4 pad 2: +3V3 -> I2C_PWR
- Q2 pad 3: /Microcontroller/LIGHT_PWR -> I2C_PWR
- R17 pad 1: /Microcontroller/LIGHT_PWR -> I2C_PWR
- R18 pad 1: /Microcontroller/LIGHT_PWR -> I2C_PWR
- R3 pad 1: +3V3 -> I2C_PWR
- R37 pad 2: DB_LED -> /Battery Charger/BAT
- R38 pad 1: DB_LED -> /Battery Charger/BAT
- R7 pad 2: /Battery Charger/VUSB -> /Microcontroller/PUMP_DRIVE
- R8 pad 2: Net-(IC3-3V3) -> +3V3
Routing:
- net I2C_PWR: track 0.00 -> 89.4 mm, vias 0 -> 6
- net +3V3: track 106.1 -> 59.7 mm, vias 7 -> 6
- net /Microcontroller/LIGHT_PWR: track 39.5 -> 0.00 mm, vias 3 -> 0
- net Net-(J3-1.1): track 0.00 -> 23.7 mm
- net Net-(Q1-Pad3): track 20.7 -> 2.55 mm
- net VDD: track 70.4 -> 53.1 mm
- net /Battery Charger/VUSB: track 41.4 -> 28.0 mm, vias 5 -> 3
- net Net-(IC3-3V3): track 11.7 -> 0.00 mm
- net /Microcontroller/PUMP_DRIVE: track 12.9 -> 21.8 mm, vias 0 -> 2
- net /Battery Charger/BAT: track 0.00 -> 8.12 mm, vias 0 -> 2
- net Net-(Q3-G): track 0.00 -> 4.12 mm
- net DB_LED: track 10.6 -> 7.65 mm
- net Net-(J1-CC1): track 1.76 -> 3.70 mm
- net Net-(D2-A): track 2.54 -> 1.35 mm
- net Net-(IC1-OUT): track 3.75 -> 2.60 mm
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Other:
- board text added: "GND"
- board text added: "PHOTO SENSE"
- board text added: "| Max. Soil Level |"
- board text removed: "LIGHT SENSOR"
- board text removed: "Plant Bot"
- board text removed: "| Soil Level |"

Commit message: updated prod files with fiducials
Parts:
- added FID1: Fiducial, personal:Product Stamp, B.Cu at (226.2, 121.5)
- added FID2: Fiducial, personal:jlcpcb_logo_2mm, B.Cu at (215.3, 86.7)
- moved ? 37.2 mm to (212.9, 124.5)
